File: relay_board/DipSwitch.kicad_sch (KiCad schematic)
At the start: 28 parts, among them SW1 SW_DIP_x06, U1 MCP23008-xSO, U2 MCP2562, U9 PIC18F26K83

Commit message: Changed to Hierarchical labels and added reverse voltage protection. Still need to do resistor math for voltage protection.
Parts:
- added D10, D11, D12, D13, D14, D15: D, Diode_SMD:D_SMB_Handsoldering, symbol Device:D
- added R39, R40, R41, R42, R43, R44: 10K, Resistor_SMD:R_0805_2012Metric_Pad1.20x1.40mm_HandSolder, symbol Device:R_US
Connections:
- net +5V: now also D11.1 (K), D13.1 (K), D14.1 (K)
- net GND: now also D10.2 (A), D12.2 (A), D15.2 (A)
- net VSENSE_BATTERY: now also R40.2; no longer U9.23 (RB2)
- net VSENSE_OUTPUT1: now also R43.1; no longer U9.7 (RA5)
- net VSENSE_OUTPUT2: now also R39.2; no longer U9.16 (RC5)
- new net: R42.1, U9.23 (RB2)
- new net: D12.1 (K), D13.2 (A), R40.1, R42.2
- new net: R41.1, U9.16 (RC5)
- new net: D10.1 (K), D11.2 (A), R39.1, R41.2
- new net: D14.2 (A), D15.1 (K), R43.2, R44.1
- new net: R44.2, U9.7 (RA5)

Commit message: Finished Reverse Voltage Math, added labels
Parts:
- D10, D11, D12, D13, D14, D15: value D -> 1N5819W
- R39, R40, R43: value 10K -> 47R
Other:
- note added: "6 PIN DIP SWITCH"
- note added: "CAN TRANSCEIVER"
- note added: "Diode Resistance Value V = IR 40V = 1A(R) R = 47R in E12 Series"
- note added: "I/O EXPANDER"
- note added: "MICROCONTROLLER"
- moved on the sheet: D14, R15, R16, R17, R18, R19, R20, R39, R40, SW1

Commit message: requested changes 1
Parts:
- D10, D11, D12, D13, D14, D15: footprint Diode_SMD:D_SMB_Handsoldering -> relay_board:SODFL3618X110N
Changed lines of the file:
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@@
 			)
 		)
-		(property "Footprint" "Diode_SMD:D_SMB_Handsoldering"
+		(property "Footprint" "relay_board:SODFL3618X110N"
 			(at 198.12 80.01 0)
 			(effects
@@
 			)
 		)
-		(property "Datasheet" "~"
+		(property "Datasheet" "https://www.smc-diodes.com/propdf/1N5817W%20THRU%201N5819W%20N1756%20REV.A.pdf"
 			(at 198.12 80.01 0)
 			(effects
@@
 			)
 		)
-		(property "Datasheet" ""
+		(property "Datasheet" "https://ww1.microchip.com/downloads/en/DeviceDoc/PIC18(L)F2526K83-Data-Sheet-DS40001943C.pdf"
 			(at 127 88.9 0)
 			(effects
@@
 			)
 		)
-		(property "Footprint" "Diode_SMD:D_SMB_Handsoldering"
+		(property "Footprint" "relay_board:SODFL3618X110N"
 			(at 173.99 105.41 0)
 			(effects
@@
 			)
 		)
-		(property "Datasheet" "~"
+		(property "Datasheet" "https://www.smc-diodes.com/propdf/1N5817W%20THRU%201N5819W%20N1756%20REV.A.pdf"
 			(at 173.99 105.41 0)
 			(effects
@@
 			)
 		)
-		(property "Datasheet" ""
+		(property "Datasheet" "https://ww1.microchip.com/downloads/en/DeviceDoc/20005167C.pdf"
 			(at 251.46 138.43 0)
 			(effects
@@
 			)
 		)
-		(property "Footprint" "Diode_SMD:D_SMB_Handsoldering"
+		(property "Footprint" "relay_board:SODFL3618X110N"
 			(at 29.21 60.96 0)
 			(effects
@@
 			)
 		)
-		(property "Datasheet" "~"
+		(property "Datasheet" "https://www.smc-diodes.com/propdf/1N5817W%20THRU%201N5819W%20N1756%20REV.A.pdf"
 			(at 29.21 60.96 0)
 			(effects
@@
 			)
 		)
-		(property "Footprint" "Diode_SMD:D_SMB_Handsoldering"
+		(property "Footprint" "relay_board:SODFL3618X110N"
 			(at 40.64 104.14 0)
 			(effects
@@
 			)
 		)
-		(property "Datasheet" "~"
+		(property "Datasheet" "https://www.smc-diodes.com/propdf/1N5817W%20THRU%201N5819W%20N1756%20REV.A.pdf"
 			(at 40.64 104.14 0)
 			(effects
@@
 			)
 		)
-		(property "Footprint" "Diode_SMD:D_SMB_Handsoldering"
+		(property "Footprint" "relay_board:SODFL3618X110N"
 			(at 198.12 95.25 0)
 			(effects
@@
 			)
 		)
-		(property "Datasheet" "~"
+		(property "Datasheet" "https://www.smc-diodes.com/propdf/1N5817W%20THRU%201N5819W%20N1756%20REV.A.pdf"
 			(at 198.12 95.25 0)
 			(effects
@@
 			)
 		)
-		(property "Footprint" "Diode_SMD:D_SMB_Handsoldering"
+		(property "Footprint" "relay_board:SODFL3618X110N"
 			(at 173.99 120.65 0)
 			(effects
@@
 			)
 		)
-		(property "Datasheet" "~"
+		(property "Datasheet" "https://www.smc-diodes.com/propdf/1N5817W%20THRU%201N5819W%20N1756%20REV.A.pdf"
 			(at 173.99 120.65 0)
 			(effects

Commit message: fix symbols; routing v1
Parts:
- removed R29, R32, R34: 10K, Resistor_SMD:R_0805_2012Metric_Pad1.20x1.40mm_HandSolder, symbol Device:R_US
- removed R30, R31, R33: DNP, Resistor_SMD:R_0805_2012Metric_Pad1.20x1.40mm_HandSolder, symbol Device:R_US
- added R21: 20K, Resistor_SMD:R_0805_2012Metric_Pad1.20x1.40mm_HandSolder, symbol Device:R_US
- added R22: 10K, Resistor_SMD:R_0805_2012Metric_Pad1.20x1.40mm_HandSolder, symbol Device:R_US
- D10, D11, D12, D13, D14, D15: footprint relay_board:SODFL3618X110N -> Diode_SMD:D_SOD-123
- U1: value MCP23008-xSO -> MCP23008
Connections:
- net CURR_SENSE_2: now also U9.16 (RC5); no longer U9.17 (RC6)
- net GND: now also U1.3 (A2), U1.4 (A1), U1.5 (A0), R22.1
- net VSENSE_12V: now also R21.2, R22.2
- net at R41.1: now also U9.17 (RC6); no longer U9.16 (RC5)
- new net +12V: R21.1
Other:
- note added: "= 12(10K/(20K+10K)) = 12/3 = 4V"
- moved on the sheet: C4, R1, R2, U1
