File: clientside_board/5v_power.kicad_sch (KiCad schematic)
At the start: 14 parts, among them U11 TPS54308, U7 INA180A3

Commit message: Top sheet update
Parts:
- C33: renamed from C34; footprint (none) -> Capacitor_SMD:C_0603_1608Metric_Pad1.08x0.95mm_HandSolder
- C34: renamed from C36; footprint (none) -> Capacitor_SMD:C_0603_1608Metric_Pad1.08x0.95mm_HandSolder
- C35: renamed from C26; footprint Capacitor_SMD:C_0805_2012Metric_Pad1.18x1.45mm_HandSolder -> Capacitor_SMD:C_0603_1608Metric_Pad1.08x0.95mm_HandSolder
- C36: renamed from C35; footprint (none) -> Capacitor_SMD:C_0603_1608Metric_Pad1.08x0.95mm_HandSolder
- renumbered R52 to R50, R39 to R51, R50 to R52, R51 to R53, U11 to U10, U7 to U11
Changed lines of the file:
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@@
 		(dnp no)
 		(fields_autoplaced yes)
-		(property "Reference" "#PWR0155"
+		(property "Reference" "#PWR0151"
 			(at 138.43 67.31 0)
 			(effects
@@
 			(project ""
 				(path "/94506b77-3097-414f-927c-35c0af27646f/60ef00a2-ee56-485c-b6f7-d62c1ab7653f"
-					(reference "#PWR0155")
+					(reference "#PWR0151")
 					(unit 1)
 				)
@@
 		(dnp no)
 		(fields_autoplaced yes)
-		(property "Reference" "R52"
+		(property "Reference" "R50"
 			(at 115.57 129.5399 0)
 			(effects
@@
 			(project "clientside_board"
 				(path "/94506b77-3097-414f-927c-35c0af27646f/60ef00a2-ee56-485c-b6f7-d62c1ab7653f"
-					(reference "R52")
+					(reference "R50")
 					(unit 1)
 				)
@@
 		(dnp no)
 		(fields_autoplaced yes)
-		(property "Reference" "#PWR0154"
+		(property "Reference" "#PWR0149"
 			(at 106.68 67.31 0)
 			(effects
@@
 			(project ""
 				(path "/94506b77-3097-414f-927c-35c0af27646f/60ef00a2-ee56-485c-b6f7-d62c1ab7653f"
-					(reference "#PWR0154")
+					(reference "#PWR0149")
 					(unit 1)
 				)
@@
 		(dnp no)
 		(fields_autoplaced yes)
-		(property "Reference" "R51"
+		(property "Reference" "R53"
 			(at 180.34 64.7699 0)
 			(effects
@@
 			(project ""
 				(path "/94506b77-3097-414f-927c-35c0af27646f/60ef00a2-ee56-485c-b6f7-d62c1ab7653f"
-					(reference "R51")
+					(reference "R53")
 					(unit 1)
 				)
@@
 		(on_board yes)
 		(dnp no)
-		(property "Reference" "#PWR0116"
+		(property "Reference" "#PWR0153"
 			(at 163.83 133.35 0)
 			(effects
@@
 			(project "clientside_board"
 				(path "/94506b77-3097-414f-927c-35c0af27646f/60ef00a2-ee56-485c-b6f7-d62c1ab7653f"
-					(reference "#PWR0116")
+					(reference "#PWR0153")
 					(unit 1)
 				)
@@
 		(dnp no)
 		(fields_autoplaced yes)
-		(property "Reference" "U11"
+		(property "Reference" "U10"
 			(at 138.43 39.37 0)
 			(effects
@@
 			(project ""
 				(path "/94506b77-3097-414f-927c-35c0af27646f/60ef00a2-ee56-485c-b6f7-d62c1ab7653f"
-					(reference "U11")
+					(reference "U10")
 					(unit 1)
 				)
@@
 		(dnp no)
 		(fields_autoplaced yes)
-		(property "Reference" "#PWR0152"
+		(property "Reference" "#PWR0150"
 			(at 113.03 151.13 0)
 			(effects
@@
 			(project "clientside_board"
 				(path "/94506b77-3097-414f-927c-35c0af27646f/60ef00a2-ee56-485c-b6f7-d62c1ab7653f"
-					(reference "#PWR0152")
+					(reference "#PWR0150")
 					(unit 1)
 				)
@@
 		(on_board yes)
 		(dnp no)
-		(property "Reference" "U7"
+		(property "Reference" "U11"
 			(at 166.37 152.4 0)
 			(effects
@@
 			(project "clientside_board"
 				(path "/94506b77-3097-414f-927c-35c0af27646f/60ef00a2-ee56-485c-b6f7-d62c1ab7653f"
-					(reference "U7")
+					(reference "U11")
 					(unit 1)
 				)
@@
 		(dnp no)
 		(fields_autoplaced yes)
-		(property "Reference" "C36"
+		(property "Reference" "C34"
 			(at 157.48 35.56 90)
 			(effects
@@
 			)
 		)
-		(property "Footprint" ""
+		(property "Footprint" "Capacitor_SMD:C_0603_1608Metric_Pad1.08x0.95mm_HandSolder"
 			(at 161.29 42.2148 0)
 			(effects
@@
 			(project ""
 				(path "/94506b77-3097-414f-927c-35c0af27646f/60ef00a2-ee56-485c-b6f7-d62c1ab7653f"
-					(reference "C36")
+					(reference "C34")
 					(unit 1)
 				)
@@
 		(on_board yes)
 		(dnp no)
-		(property "Reference" "C26"
+		(property "Reference" "C35"
 			(at 172.72 137.1133 90)
 			(effects
@@
 			)
 		)
-		(property "Footprint" "Capacitor_SMD:C_0805_2012Metric_Pad1.18x1.45mm_HandSolder"
+		(property "Footprint" "Capacitor_SMD:C_0603_1608Metric_Pad1.08x0.95mm_HandSolder"
 			(at 176.53 131.7752 0)
 			(effects
@@
 			(project "clientside_board"
 				(path "/94506b77-3097-414f-927c-35c0af27646f/60ef00a2-ee56-485c-b6f7-d62c1ab7653f"
-					(reference "C26")
+					(reference "C35")
 					(unit 1)
 				)
@@
 		(dnp no)
 		(fields_autoplaced yes)
-		(property "Reference" "#PWR0146"
+		(property "Reference" "#PWR0157"
 			(at 201.93 124.46 0)
 			(effects
@@
 			(project ""
 				(path "/94506b77-3097-414f-927c-35c0af27646f/60ef00a2-ee56-485c-b6f7-d62c1ab7653f"
-					(reference "#PWR0146")
+					(reference "#PWR0157")
 					(unit 1)
 				)
@@
 		(dnp no)
 		(fields_autoplaced yes)
-		(property "Reference" "C34"
+		(property "Reference" "C33"
 			(at 110.49 52.0699 0)
 			(effects
@@
 			)
 		)
-		(property "Footprint" ""
+		(property "Footprint" "Capacitor_SMD:C_0603_1608Metric_Pad1.08x0.95mm_HandSolder"
 			(at 107.6452 57.15 0)
 			(effects
@@
 			(project ""
 				(path "/94506b77-3097-414f-927c-35c0af27646f/60ef00a2-ee56-485c-b6f7-d62c1ab7653f"
-					(reference "C34")
+					(reference "C33")
 					(unit 1)
 				)
@@
 		(dnp no)
 		(fields_autoplaced yes)
-		(property "Reference" "#PWR0118"
+		(property "Reference" "#PWR0155"
 			(at 179.07 139.7 0)
 			(effects
@@
 			(project "clientside_board"
 				(path "/94506b77-3097-414f-927c-35c0af27646f/60ef00a2-ee56-485c-b6f7-d62c1ab7653f"
-					(reference "#PWR0118")
+					(reference "#PWR0155")
 					(unit 1)
 				)
@@
 		(dnp no)
 		(fields_autoplaced yes)
-		(property "Reference" "C35"
+		(property "Reference" "C36"
 			(at 203.2 58.4199 0)
 			(effects
@@
 			)
 		)
-		(property "Footprint" ""
+		(property "Footprint" "Capacitor_SMD:C_0603_1608Metric_Pad1.08x0.95mm_HandSolder"
 			(at 200.3552 63.5 0)
 			(effects
@@
 			(project ""
 				(path "/94506b77-3097-414f-927c-35c0af27646f/60ef00a2-ee56-485c-b6f7-d62c1ab7653f"
-					(reference "C35")
+					(reference "C36")
 					(unit 1)
 				)
@@
 		(dnp no)
 		(fields_autoplaced yes)
-		(property "Reference" "R50"
+		(property "Reference" "R52"
 			(at 180.34 54.6099 0)
 			(effects
@@
 			(project ""
 				(path "/94506b77-3097-414f-927c-35c0af27646f/60ef00a2-ee56-485c-b6f7-d62c1ab7653f"
-					(reference "R50")
+					(reference "R52")
 					(unit 1)
 				)
@@
 		(dnp no)
 		(fields_autoplaced yes)
-		(property "Reference" "#PWR0114"
+		(property "Reference" "#PWR0152"
 			(at 151.13 166.37 0)
 			(effects
@@
 			(project "clientside_board"
 				(path "/94506b77-3097-414f-927c-35c0af27646f/60ef00a2-ee56-485c-b6f7-d62c1ab7653f"
-					(reference "#PWR0114")
+					(reference "#PWR0152")
 					(unit 1)
 				)
@@
 		(dnp no)
 		(fields_autoplaced yes)
-		(property "Reference" "#PWR0153"
+		(property "Reference" "#PWR0148"
 			(at 96.52 46.99 0)
 			(effects
@@
 			(project ""
 				(path "/94506b77-3097-414f-927c-35c0af27646f/60ef00a2-ee56-485c-b6f7-d62c1ab7653f"
-					(reference "#PWR0153")
+					(reference "#PWR0148")
 					(unit 1)
 				)
@@
 		(dnp no)
 		(fields_autoplaced yes)
-		(property "Reference" "R39"
+		(property "Reference" "R51"
 			(at 146.05 119.4267 90)
 			(effects
@@
 			(project "clientside_board"
 				(path "/94506b77-3097-414f-927c-35c0af27646f/60ef00a2-ee56-485c-b6f7-d62c1ab7653f"
-					(reference "R39")
+					(reference "R51")
 					(unit 1)
 				)
@@
 		(dnp no)
 		(fields_autoplaced yes)
-		(property "Reference" "#PWR0151"
+		(property "Reference" "#PWR0154"
 			(at 177.8 78.74 0)
 			(effects
@@
 			(project ""
 				(path "/94506b77-3097-414f-927c-35c0af27646f/60ef00a2-ee56-485c-b6f7-d62c1ab7653f"
-					(reference "#PWR0151")
-					(unit 1)
-				)
+					(reference "#PWR0154")
+					(unit 1)
+				)
